File: boards/bench-psu/hardware/kicad/bench-psu.kicad_sch (KiCad schematic)
At the start: 87 parts, among them J1 TYPE-C 16PIN 2MD(073), J2 DG301-5.0-04P-14-1000A(H), J3 PZ254V-11-04P, J4 PZ254V-11-05P, Q1 AO4407A, SW1 TS-1187A-B-A-B, SW2 TS-1187A-B-A-B, U1 STUSB4500QTR, U11 LMR51635YDDCR, U12 INA219AIDCNR, U2 USBLC6-2SC6, U21 LMR51635YDDCR, U22 INA219AIDCNR, U3 LMR51635YDDCR, U4 AP2112K-3.3TRG1, U5 ESP32-S3-MINI-1-N8

Commit message: bench-psu rev B: LMR33630 bucks, INA226 with hardware over-current trip, fail-safe FB current sink
- Converter: LMR33630A (400 kHz, 3 A) per channel and for the 5 V rail; FXL1040 10 uH inductor
- Voltage set: TLV9062 + NPN current sink on FB (1.6 V at 0 V/floating PWM, 16.6 V max)
- Loop compensation: 6.8k + 220 nF lag network on FB (simulated PM 52-75 deg)
- Measurement: INA226 on 20 mR shunt; ALERT pulls buck EN low (hardware trip)
- Input: SMBJ22A TVS, gate divider for AO4407A Vgs, SMD electrolytic
- Add SPICE sim decks, scripts, plots (boards/bench-psu/sim)
- Regenerate review set and fab files; update README

Co-Authored-By: Claude Opus 5.5 <noreply@anthropic.com>
Parts:
- added C112: 100nF, tscircuit:capacitor_cap0603, symbol vibepcb:C112
- added C113: 220nF, tscircuit:capacitor_cap0603, symbol vibepcb:C113
- added C19: 100nF, tscircuit:capacitor_cap0603, symbol vibepcb:C19
- added C20: 1uF, tscircuit:capacitor_cap0603, symbol vibepcb:C20
- added C21: 100nF, tscircuit:capacitor_cap0603, symbol vibepcb:C21
- added C212: 100nF, tscircuit:capacitor_cap0603, symbol vibepcb:C212
- added C213: 220nF, tscircuit:capacitor_cap0603, symbol vibepcb:C213
- added Q11: MMBT3904(RANGE:100-300), tscircuit:MMBT3904_RANGE_100-300, symbol vibepcb:Q11
- added Q21: MMBT3904(RANGE:100-300), tscircuit:MMBT3904_RANGE_100-300, symbol vibepcb:Q21
- added R109: 100kΩ, tscircuit:resistor_res0603, symbol vibepcb:R109
- added R110: 10kΩ, tscircuit:resistor_res0603, symbol vibepcb:R110
- added R111: 6.8kΩ, tscircuit:resistor_res0603, symbol vibepcb:R111
- added R209: 100kΩ, tscircuit:resistor_res0603, symbol vibepcb:R209
- added R210: 10kΩ, tscircuit:resistor_res0603, symbol vibepcb:R210
- added R211: 6.8kΩ, tscircuit:resistor_res0603, symbol vibepcb:R211
- added R7: 47kΩ, tscircuit:resistor_res0603, symbol vibepcb:R7
- added U6: TLV9062IDR, tscircuit:TLV9062IDR, symbol vibepcb:U6
- C10, C103, C203: footprint tscircuit:capacitor_cap0805 -> tscircuit:capacitor_cap0603; LCSC C28233 -> C14663
- C101, C102, C201, C202, C7, C8, C9: value 2.2uF -> 10uF; LCSC C170101 -> C13585
- C105, C205: value 4.7uF -> 1uF; footprint tscircuit:capacitor_cap1210 -> tscircuit:capacitor_cap0603; LCSC C337978 -> C15849
- C106, C107, C206, C207: value 4.7uF -> 22uF; footprint tscircuit:capacitor_cap1210 -> tscircuit:capacitor_cap1206; LCSC C337978 -> C12891
- C108, C208: value 100nF -> 22uF; footprint tscircuit:capacitor_cap0603 -> tscircuit:capacitor_cap1206; LCSC C14663 -> C12891
- C109, C209: value 100uF -> 22uF; footprint tscircuit:NXA63V100M8_15_LO -> tscircuit:capacitor_cap1206; LCSC C3002361 -> C12891; MPN NXA63V100M8*15 LO -> (none)
- C6: footprint tscircuit:NXA63V100M8_15_LO -> tscircuit:RVT1V101M0607_100UF_35V; LCSC C3002361 -> C970686; MPN NXA63V100M8*15 LO -> RVT1V101M0607 100UF 35V
- D1: value SMBJ24A -> SMBJ22A; footprint tscircuit:SMBJ24A -> tscircuit:SMBJ22A; LCSC C123819 -> C151920; MPN SMBJ24A -> SMBJ22A
- L1: value 10µH -> 15µH; footprint tscircuit:SWPA6045S100MT -> tscircuit:SWPA4030S150MT; LCSC C79272 -> C83475; MPN SWPA6045S100MT -> SWPA4030S150MT
- L11, L21: footprint tscircuit:SWPA6045S100MT -> tscircuit:FXL1040-100-M; LCSC C79272 -> C475915; MPN SWPA6045S100MT -> FXL1040-100-M
- R101, R201: value 100mΩ -> 20mΩ; LCSC C500724 -> C105360
- R102, R202: value 100kΩ -> 120kΩ; LCSC C25803 -> C25808
- R103, R203: value 12kΩ -> 200kΩ; LCSC C22790 -> C25811
- R104, R204: value 12kΩ -> 2.4kΩ; LCSC C22790 -> C22940
- R105, R205: value 20kΩ -> 1kΩ; LCSC C4184 -> C21190
- R107, R207: value 10kΩ -> 100kΩ; LCSC C25804 -> C25803
- R108, R208: value 100kΩ -> 10kΩ; LCSC C25803 -> C25804
- R6: value 20kΩ -> 24kΩ; LCSC C4184 -> C23352
- U11, U21, U3: value LMR51635YDDCR -> LMR33630ADDAR; footprint tscircuit:LMR51635YDDCR -> tscircuit:LMR33630ADDAR; LCSC C45262770 -> C841384; MPN LMR51635YDDCR -> LMR33630ADDAR
- U12, U22: value INA219AIDCNR -> INA226AIDGSR; footprint tscircuit:INA219AIDCNR -> tscircuit:INA226AIDGSR; LCSC C87469 -> C49851; MPN INA219AIDCNR -> INA226AIDGSR
Connections:
- net EN1: now also U11.3 (EN), U12.3 (~{Alert}), R109.1 (pin1), R110.2 (pin2); no longer R108.1 (pin1), U11.2 (EN), U5.10 (IO6)
- net EN2: now also U21.3 (EN), U22.3 (~{Alert}), R209.1 (pin1), R210.2 (pin2); no longer R208.1 (pin1), U21.2 (EN), U5.11 (IO7)
- net FB1: now also U11.5 (FB), Q11.3 (C), R111.1 (pin1); no longer R104.1 (pin1), R105.1 (pin1), U11.1 (FB)
- net FB2: now also U21.5 (FB), Q21.3 (C), R211.1 (pin1); no longer R204.1 (pin1), R205.1 (pin1), U21.1 (FB)
- net FB5: now also U3.5 (FB); no longer U3.1 (FB)
- net GND: now also U11.1 (GND), U11.9 (GND), U12.1 (A1), U12.2 (A0), U21.1 (GND), U21.9 (GND), U22.1 (A1), U22.7 (GND), U3.1 (GND), U3.9 (GND), C112.2 (pin2), C113.2 (pin2), C20.2 (pin2), C21.2 (pin2), C212.2 (pin2), C213.2 (pin2), R109.2 (pin2), R209.2 (pin2), U6.4 (VEE/GND); no longer U11.4 (GND), U12.3 (GND), U12.8 (A1), U21.4 (GND), U22.3 (GND), U22.8 (A1), U3.4 (GND)
- net I2C_SDA: now also U12.4 (SDA), U22.4 (SDA); no longer U12.6 (SDA), U22.6 (SDA)
- net OUT1: now also R102.1 (pin1), U12.8 (Vbus), U12.9 (Vin-); no longer U12.2 (IN-)
- net OUT1_B: now also C108.1 (pin1), U12.10 (Vin+); no longer C105.1 (pin1), R102.1 (pin1), U12.1 (IN+)
- net OUT2: now also R202.1 (pin1), U22.8 (Vbus), U22.9 (Vin-); no longer U22.2 (IN-)
- net OUT2_B: now also C208.1 (pin1), U22.10 (Vin+); no longer C205.1 (pin1), R202.1 (pin1), U22.1 (IN+)
- net PD_GATE: now also C19.2 (pin2), R7.2 (pin2); no longer U1.16 (VBUS_EN_SNK)
- net PWM1: no longer C110.1 (pin1), R105.2 (pin2)
- net PWM2: no longer C210.1 (pin1), R205.2 (pin2)
- net SW5: now also U3.8 (SW); no longer U3.5 (SW)
- net U3_EN: now also U3.3 (EN); no longer U3.2 (EN)
- net V3V3: now also U12.6 (VS), U22.2 (A0), U22.6 (VS), C112.1 (pin1), C21.1 (pin1), C212.1 (pin1), U6.8 (VCC); no longer C108.1 (pin1), C208.1 (pin1), U12.4 (VS), U22.4 (VS), U22.7 (A0)
- net VBUS: now also C19.1 (pin1)
- net VIN: now also U11.2 (VIN), U21.2 (VIN), U3.2 (VIN); no longer U11.3 (VIN), U21.3 (VIN), U3.3 (VIN)
- net Net-(R106-Pad2) renamed PWM1_F
- net PWM1_F: now also C110.1 (pin1)
- net Net-(R107-Pad2) renamed VSET1
- net VSET1: now also R108.1 (pin1), U6.3 (INA+)
- net Net-(R206-Pad2) renamed PWM2_F
- net PWM2_F: now also C210.1 (pin1)
- net Net-(R207-Pad2) renamed VSET2
- net VSET2: now also R208.1 (pin1), U6.5 (INB+)
- net SW1 renamed SW_CH1
- net SW_CH1: now also U11.8 (SW); no longer U11.5 (SW)
- net SW2 renamed SW_CH2
- net SW_CH2: now also U21.8 (SW); no longer U21.5 (SW)
- net U11_CB renamed U11_BOOT
- net U11_BOOT: now also U11.7 (BOOT); no longer U11.6 (CB)
- net U21_CB renamed U21_BOOT
- net U21_BOOT: now also U21.7 (BOOT); no longer U21.6 (CB)
- net U3_CB renamed U3_BOOT
- net U3_BOOT: now also U3.7 (BOOT); no longer U3.6 (CB)
- new net EN1_MCU: R110.1 (pin1), U5.10 (IO6)
- new net EN2_MCU: R210.1 (pin1), U5.11 (IO7)
- new net ISET1_DRV: R105.1 (pin1), U6.1 (OUTA)
- new net ISET1_E: Q11.2 (E), R104.1 (pin1), U6.2 (INA-)
- new net ISET2_DRV: R205.1 (pin1), U6.7 (OUTB)
- new net ISET2_E: Q21.2 (E), R204.1 (pin1), U6.6 (INB-)
- new net Net-(R111-Pad2): C113.1 (pin1), R111.2 (pin2)
- new net Net-(R211-Pad2): C213.1 (pin1), R211.2 (pin2)
- new net PD_EN: R7.1 (pin1), U1.16 (VBUS_EN_SNK)
- new net Q11_B: Q11.1 (B), R105.2 (pin2)
- new net Q21_B: Q21.1 (B), R205.2 (pin2)
- new net U11_VCC: C105.1 (pin1), U11.6 (VCC)
- new net U21_VCC: C205.1 (pin1), U21.6 (VCC)
- new net U3_VCC: C20.1 (pin1), U3.6 (VCC)
- no-connect marks 36 -> 39
Other:
- moved on the sheet: C1, C10, C101, C102, C103, C104, C105, C106, C107, C108, C109, C11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

Commit message: bench-psu: output status LEDs, silkscreen pass, bring-up guide
- Per channel ON LED (KT-0603YG, driven from the buck EN node through an NPN: shows the
  hardware state, dark after an INA226 trip) and OC LED (KT-0603R on IO21 / IO47)
- Silkscreen: LED functions, header pin labels at fab-legal size, RST/BOOT and the title
  moved off parts and pads, rail probe points (VIN, 5V, 3V3), PD input label, pin and
  I2C-address summary on the back
- README: bring-up guide (unpowered checks, logic at 5 V, firmware/I2C, channels at 5 V,
  20 V), LED design notes, pin map
- Republished review set; findings.toml from the new check verification

hardware/fab (gerbers, CPL) is NOT regenerated and still shows the board without LEDs:
`pcb fab` now needs `check --strict`, which fails on the open verification items.

Co-Authored-By: Claude Opus 5.5 <noreply@anthropic.com>
Parts:
- added D101: KT-0603YG, tscircuit:KT-0603YG, symbol vibepcb:D101
- added D102: KT-0603R, tscircuit:KT-0603R, symbol vibepcb:D102
- added D201: KT-0603YG, tscircuit:KT-0603YG, symbol vibepcb:D201
- added D202: KT-0603R, tscircuit:KT-0603R, symbol vibepcb:D202
- added Q12: MMBT3904(RANGE:100-300), tscircuit:MMBT3904_RANGE_100-300, symbol vibepcb:Q12
- added Q22: MMBT3904(RANGE:100-300), tscircuit:MMBT3904_RANGE_100-300, symbol vibepcb:Q22
- added R112: 1kΩ, tscircuit:resistor_res0603, symbol vibepcb:R112
- added R113: 1kΩ, tscircuit:resistor_res0603, symbol vibepcb:R113
- added R114: 47kΩ, tscircuit:resistor_res0603, symbol vibepcb:R114
- added R212: 1kΩ, tscircuit:resistor_res0603, symbol vibepcb:R212
- added R213: 1kΩ, tscircuit:resistor_res0603, symbol vibepcb:R213
- added R214: 47kΩ, tscircuit:resistor_res0603, symbol vibepcb:R214
Connections:
- net EN1: now also R114.1 (pin1)
- net EN2: now also R214.1 (pin1)
- net GND: now also D102.2 (pin2), D202.2 (pin2), Q12.2 (E), Q22.2 (E)
- net V3V3: now also R112.1 (pin1), R212.1 (pin1)
- net LED_OC1: now reaches U5.25 (IO21)
- net LED_OC1: now also R113.1 (pin1)
- net LED_OC2: now reaches U5.27 (IO47)
- net LED_OC2: now also R213.1 (pin1)
- new net Net-(D101-Pad1): D101.1 (pin1), R112.2 (pin2)
- new net Net-(D102-Pad1): D102.1 (pin1), R113.2 (pin2)
- new net Net-(D201-Pad1): D201.1 (pin1), R212.2 (pin2)
- new net Net-(D202-Pad1): D202.1 (pin1), R213.2 (pin2)
- new net Q12_B: Q12.1 (B), R114.2 (pin2)
- new net Q12_C: D101.2 (pin2), Q12.3 (C)
- new net Q22_B: Q22.1 (B), R214.2 (pin2)
- new net Q22_C: D201.2 (pin2), Q22.3 (C)
- no-connect marks 39 -> 37
Other:
- moved on the sheet: C1, C10, C101, C102, C103, C104, C105, C106, C107, C108, C109, C11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

Commit message: clean up after rev C: hardware/ republished from rev C (stale rev B fab/ removed), sim results and loop plots regenerated from the rev C decks (rev B load-point/switching data dropped), README and sim/README rewritten for rev C (history table, six review rounds, parts bought separately, open point on the loop's mid-band phase)
Co-Authored-By: Claude Opus 5.5 <noreply@anthropic.com>
Parts:
- removed J4: PZ254V-11-05P, tscircuit:PZ254V-11-05P, symbol vibepcb:J4
- added C114: 100nF, tscircuit:capacitor_cap0603, symbol vibepcb:C114
- added C115: 100nF, tscircuit:capacitor_cap0603, symbol vibepcb:C115
- added C116: 100nF, tscircuit:capacitor_cap0603, symbol vibepcb:C116
- added C117: 100nF, tscircuit:capacitor_cap0603, symbol vibepcb:C117
- added C118: 1uF, tscircuit:capacitor_cap0603, symbol vibepcb:C118
- added C119: 100nF, tscircuit:capacitor_cap0603, symbol vibepcb:C119
- added C120: 100nF, tscircuit:capacitor_cap0603, symbol vibepcb:C120
- added C130: 33nF, tscircuit:capacitor_cap0603, symbol vibepcb:C130
- added C131: 33nF, tscircuit:capacitor_cap0603, symbol vibepcb:C131
- added C132: 33nF, tscircuit:capacitor_cap0603, symbol vibepcb:C132
- added C133: 33nF, tscircuit:capacitor_cap0603, symbol vibepcb:C133
- added C214: 100nF, tscircuit:capacitor_cap0603, symbol vibepcb:C214
- added C215: 100nF, tscircuit:capacitor_cap0603, symbol vibepcb:C215
- added C216: 100nF, tscircuit:capacitor_cap0603, symbol vibepcb:C216
- added C217: 100nF, tscircuit:capacitor_cap0603, symbol vibepcb:C217
- added C218: 1uF, tscircuit:capacitor_cap0603, symbol vibepcb:C218
- added C219: 100nF, tscircuit:capacitor_cap0603, symbol vibepcb:C219
- added C22: 100nF, tscircuit:capacitor_cap0603, symbol vibepcb:C22
- added C220: 100nF, tscircuit:capacitor_cap0603, symbol vibepcb:C220
- added C23: 22uF, tscircuit:capacitor_cap1206, symbol vibepcb:C23
- added C230: 33nF, tscircuit:capacitor_cap0603, symbol vibepcb:C230
- added C231: 33nF, tscircuit:capacitor_cap0603, symbol vibepcb:C231
- added C232: 33nF, tscircuit:capacitor_cap0603, symbol vibepcb:C232
- added C233: 33nF, tscircuit:capacitor_cap0603, symbol vibepcb:C233
- added C24: 22uF, tscircuit:capacitor_cap1206, symbol vibepcb:C24
- added C25: 100uF, tscircuit:RVT1V101M0607_100UF_35V, symbol vibepcb:C25
- added C26: 100uF, tscircuit:RVT1V101M0607_100UF_35V, symbol vibepcb:C26
- added D13: SS54, tscircuit:SS54, symbol vibepcb:D13
- added D14: 1N4148W, tscircuit:1N4148W, symbol vibepcb:D14
- added D15: 1N4148W, tscircuit:1N4148W, symbol vibepcb:D15
- added D16: 1N4148W, tscircuit:1N4148W, symbol vibepcb:D16
- added D2: ESDA25P35-1U1M, tscircuit:ESDA25P35-1U1M, symbol vibepcb:D2
- added D23: SS54, tscircuit:SS54, symbol vibepcb:D23
- added D24: 1N4148W, tscircuit:1N4148W, symbol vibepcb:D24
- added D25: 1N4148W, tscircuit:1N4148W, symbol vibepcb:D25
- added D26: 1N4148W, tscircuit:1N4148W, symbol vibepcb:D26
- added ENC1: EC11E15244B2, tscircuit:EC11E15244B2, symbol vibepcb:ENC1
- added ENC2: EC11E15244B2, tscircuit:EC11E15244B2, symbol vibepcb:ENC2
- added Q13: 2N7002, tscircuit:2N7002, symbol vibepcb:Q13
- added Q14: MMBT3904(RANGE:100-300), tscircuit:MMBT3904_RANGE_100-300, symbol vibepcb:Q14
- added Q23: 2N7002, tscircuit:2N7002, symbol vibepcb:Q23
- added Q24: MMBT3904(RANGE:100-300), tscircuit:MMBT3904_RANGE_100-300, symbol vibepcb:Q24
- added R115: 10kΩ, tscircuit:resistor_res0603, symbol vibepcb:R115
- added R116: 10kΩ, tscircuit:resistor_res0603, symbol vibepcb:R116
- added R117: 10kΩ, tscircuit:resistor_res0603, symbol vibepcb:R117
- added R118: 330Ω, tscircuit:resistor_res0603, symbol vibepcb:R118
- added R119: 10kΩ, tscircuit:resistor_res0603, symbol vibepcb:R119
- added R120: 100kΩ, tscircuit:resistor_res0603, symbol vibepcb:R120
- added R121: 4.7kΩ, tscircuit:resistor_res0603, symbol vibepcb:R121
- added R122: 47kΩ, tscircuit:resistor_res0603, symbol vibepcb:R122
- added R123: 47kΩ, tscircuit:resistor_res0603, symbol vibepcb:R123
- added R124: 10kΩ, tscircuit:resistor_res0603, symbol vibepcb:R124
- added R125: 330Ω, tscircuit:resistor_res0603, symbol vibepcb:R125
- added R126: 100kΩ, tscircuit:resistor_res0603, symbol vibepcb:R126
- added R130: 3.3kΩ, tscircuit:resistor_res0603, symbol vibepcb:R130
- added R131: 3.3kΩ, tscircuit:resistor_res0603, symbol vibepcb:R131
- added R132: 3.3kΩ, tscircuit:resistor_res0603, symbol vibepcb:R132
- added R133: 3.3kΩ, tscircuit:resistor_res0603, symbol vibepcb:R133
- added R215: 10kΩ, tscircuit:resistor_res0603, symbol vibepcb:R215
- added R216: 10kΩ, tscircuit:resistor_res0603, symbol vibepcb:R216
- added R217: 10kΩ, tscircuit:resistor_res0603, symbol vibepcb:R217
- added R218: 330Ω, tscircuit:resistor_res0603, symbol vibepcb:R218
- added R219: 10kΩ, tscircuit:resistor_res0603, symbol vibepcb:R219
- added R220: 100kΩ, tscircuit:resistor_res0603, symbol vibepcb:R220
- added R221: 4.7kΩ, tscircuit:resistor_res0603, symbol vibepcb:R221
- added R222: 47kΩ, tscircuit:resistor_res0603, symbol vibepcb:R222
- added R223: 47kΩ, tscircuit:resistor_res0603, symbol vibepcb:R223
- added R224: 10kΩ, tscircuit:resistor_res0603, symbol vibepcb:R224
- added R225: 330Ω, tscircuit:resistor_res0603, symbol vibepcb:R225
- added R226: 100kΩ, tscircuit:resistor_res0603, symbol vibepcb:R226
- added R230: 3.3kΩ, tscircuit:resistor_res0603, symbol vibepcb:R230
- added R231: 3.3kΩ, tscircuit:resistor_res0603, symbol vibepcb:R231
- added R232: 3.3kΩ, tscircuit:resistor_res0603, symbol vibepcb:R232
- added R233: 3.3kΩ, tscircuit:resistor_res0603, symbol vibepcb:R233
- added SW13: B3F-4055, tscircuit:B3F-4055, symbol vibepcb:SW13
- added SW23: B3F-4055, tscircuit:B3F-4055, symbol vibepcb:SW23
- added TH11: 10kΩ, tscircuit:NCP18XH103F03RB, symbol vibepcb:TH11
- added TH21: 10kΩ, tscircuit:NCP18XH103F03RB, symbol vibepcb:TH21
- added TP1: test_point_smtpad_circle_d1, tscircuit:test_point_smtpad_circle_d1, symbol vibepcb:TP1
- added TP2: test_point_smtpad_circle_d1, tscircuit:test_point_smtpad_circle_d1, symbol vibepcb:TP2
- added TP3: test_point_smtpad_circle_d1, tscircuit:test_point_smtpad_circle_d1, symbol vibepcb:TP3
- added TP4: test_point_smtpad_circle_d1, tscircuit:test_point_smtpad_circle_d1, symbol vibepcb:TP4
- added TP5: test_point_smtpad_circle_d1, tscircuit:test_point_smtpad_circle_d1, symbol vibepcb:TP5
- added U13: INA181A2IDBVR, tscircuit:INA181A2IDBVR, symbol vibepcb:U13
- added U23: INA181A2IDBVR, tscircuit:INA181A2IDBVR, symbol vibepcb:U23
- added U7: TLV9062IDR, tscircuit:TLV9062IDR, symbol vibepcb:U7
- added U8: ESDA25W, tscircuit:ESDA25W, symbol vibepcb:U8
- C10, C103, C203: value 100nF -> 220nF; LCSC C14663 -> C107083
- C5: footprint tscircuit:capacitor_cap0603 -> tscircuit:capacitor_cap0805; LCSC C53987 -> C565695
- L1: value 15µH -> 6.8µH; footprint tscircuit:SWPA4030S150MT -> tscircuit:FXL0530-6R8-M; LCSC C83475 -> C177249; MPN SWPA4030S150MT -> FXL0530-6R8-M
- L11, L21: value 10µH -> 15µH; footprint tscircuit:FXL1040-100-M -> tscircuit:FXL1040-150-M; LCSC C475915 -> C475916; MPN FXL1040-100-M -> FXL1040-150-M
- R104, R204: value 2.4kΩ -> 2.2kΩ; LCSC C22940 -> C4190
Connections:
- net CC1: now also U8.1 (K)
- net CC2: now also U8.2 (K)
- net EN1: now also R122.1 (pin1)
- net EN2: now also R222.1 (pin1)
- net FB1: now also D14.1 (cathode), D16.2 (anode)
- net FB2: now also D24.1 (cathode), D26.2 (anode)
- net GND: now also C114.2 (pin2), C115.2 (pin2), C118.2 (pin2), C119.2 (pin2), C120.2 (pin2), C130.2 (pin2), C131.2 (pin2), C132.2 (pin2), C133.2 (pin2), C214.2 (pin2), C215.2 (pin2), C218.2 (pin2), C219.2 (pin2), C22.2 (pin2), C220.2 (pin2), C23.2 (pin2), C230.2 (pin2), C231.2 (pin2), C232.2 (pin2), C233.2 (pin2), C24.2 (pin2), C25.2 (pin2), C26.2 (pin2), D13.1 (anode), D2.2, D23.1 (anode), ENC1.11 (D), ENC1.6 (pin6), ENC1.7 (pin7), ENC1.9 (C), ENC2.11 (D), ENC2.6 (pin6), ENC2.7 (pin7), ENC2.9 (C), Q13.2 (S), Q14.2 (E), Q23.2 (S), Q24.2 (E), R125.2 (pin2), R225.2 (pin2), SW13.4, SW23.4, TH11.2 (pin2), TH21.2 (pin2), TP5.1 (pin1), U13.2 (GND), U13.5 (REF), U23.2 (GND), U23.5 (REF), U7.4 (VEE/GND), U8.3 (A)
- net OUT1: now also C114.1 (pin1), C25.1 (pin1), D13.2 (cathode), R121.2 (pin2), U13.4 (-)
- net OUT1_B: now also U13.3 (+)
- net OUT2: now also C214.1 (pin1), C26.1 (pin1), D23.2 (cathode), R221.2 (pin2), U23.4 (-)
- net OUT2_B: now also U23.3 (+)
- net USB_DN: now also U2.3 (I/O2), U2.4 (I/O2); no longer U2.1 (I/O1), U2.6 (I/O1)
- net USB_DP: now also U2.1 (I/O1), U2.6 (I/O1); no longer U2.3 (I/O2), U2.4 (I/O2)
- net V3V3: now also C115.1 (pin1), C215.1 (pin1), C22.1 (pin1), D16.1 (cathode), D26.1 (cathode), R124.1 (pin1), R130.1 (pin1), R131.1 (pin1), R132.1 (pin1), R133.1 (pin1), R224.1 (pin1), R230.1 (pin1), R231.1 (pin1), R232.1 (pin1), R233.1 (pin1), TP4.1 (pin1), U13.6 (V+), U23.6 (V+), U7.8 (VCC)
- net V5: now also C23.1 (pin1), C24.1 (pin1), R123.2 (pin2), R223.2 (pin2), TP3.1 (pin1)
- net VBUS: now also D2.1, TP1.1 (pin1)
- net VIN: now also TP2.1 (pin1)
- net ISET1: now reaches U5.15 (IO11)
- net ISET1: now also R119.1 (pin1)
- net ISET2: now reaches U5.16 (IO12)
- net ISET2: now also R219.1 (pin1)
- net ENC2_A: now reaches U5.17 (IO13)
- net ENC2_A: now also C230.1 (pin1), ENC2.8 (A), R230.2 (pin2)
- net ENC2_B: now reaches U5.18 (IO14)
- net ENC2_B: now also C231.1 (pin1), ENC2.10 (B), R231.2 (pin2)
- net ENC2_SW: now reaches U5.22 (IO18)
- net ENC2_SW: now also C232.1 (pin1), ENC2.12 (E), R232.2 (pin2)
- net BTN1: now reaches U5.34 (IO38)
- net BTN1: now also C133.1 (pin1), R133.2 (pin2), SW13.1
- net BTN2: now reaches U5.35 (IO39)
- net BTN2: now also C233.1 (pin1), R233.2 (pin2), SW23.1
- net NTC1: now reaches U5.5 (IO1)
- net NTC1: now also C120.1 (pin1), R124.2 (pin2), TH11.1 (pin1)
- net NTC2: now reaches U5.6 (IO2)
- net NTC2: now also C220.1 (pin1), R224.2 (pin2), TH21.1 (pin1)
- net ENC_A renamed ENC1_A
- net ENC1_A: now also C130.1 (pin1), ENC1.8 (A), R130.2 (pin2)
- net ENC_B renamed ENC1_B
- net ENC1_B: now also C131.1 (pin1), ENC1.10 (B), R131.2 (pin2)
- net ENC_SW renamed ENC1_SW
- net ENC1_SW: now also C132.1 (pin1), ENC1.12 (E), R132.2 (pin2)
- net ISET1_DRV renamed ISINK1_DRV
- net ISET1_E renamed ISINK1_E
- net ISET2_DRV renamed ISINK2_DRV
- net ISET2_E renamed ISINK2_E
- net LED_OC1 renamed LED_CC1
- net LED_OC2 renamed LED_CC2
- net Net-(R111-Pad2) renamed LAG1
- net LAG1: now also R126.2 (pin2)
- net Net-(R211-Pad2) renamed LAG2
- net LAG2: now also R226.2 (pin2)
- new net CC1_NEG: C117.1 (pin1), R117.2 (pin2), U7.2 (INA-)
- new net CC1_OUT: R116.1 (pin1), R118.2 (pin2), U7.1 (OUTA)
- new net CC2_NEG: C217.1 (pin1), R217.2 (pin2), U7.6 (INB-)
- new net CC2_OUT: R216.1 (pin1), R218.2 (pin2), U7.7 (OUTB)
- new net DIS1_G: D15.2 (anode), Q13.1 (G), Q14.3 (C), R123.1 (pin1)
- new net DIS2_G: D25.2 (anode), Q23.1 (G), Q24.3 (C), R223.1 (pin1)
- new net ISENS1: R115.1 (pin1), U13.1
- new net ISENS1_F: C116.1 (pin1), R115.2 (pin2), U7.3 (INA+)
- new net ISENS2: R215.1 (pin1), U23.1
- new net ISENS2_F: C216.1 (pin1), R215.2 (pin2), U7.5 (INB+)
- new net ISET1_A: C118.1 (pin1), R119.2 (pin2), R120.1 (pin1)
- new net ISET1_F: C119.1 (pin1), R117.1 (pin1), R120.2 (pin2)
- new net ISET2_A: C218.1 (pin1), R219.2 (pin2), R220.1 (pin1)
- new net ISET2_F: C219.1 (pin1), R217.1 (pin1), R220.2 (pin2)
- new net Net-(D15-Pad1): D15.1 (cathode), R126.1 (pin1)
- new net Net-(D25-Pad1): D25.1 (cathode), R226.1 (pin1)
- new net Net-(R116-Pad2): D14.2 (anode), R116.2 (pin2)
- new net Net-(R118-Pad1): C117.2 (pin2), R118.1 (pin1)
- new net Net-(R125-Pad1): C116.2 (pin2), R125.1 (pin1)
- new net Net-(R216-Pad2): D24.2 (anode), R216.2 (pin2)
- new net Net-(R218-Pad1): C217.2 (pin2), R218.1 (pin1)
- new net Net-(R225-Pad1): C216.2 (pin2), R225.1 (pin1)
- new net Q13_D: Q13.3 (D), R121.1 (pin1)
- new net Q14_B: Q14.1 (B), R122.2 (pin2)
- new net Q23_D: Q23.3 (D), R221.1 (pin1)
- new net Q24_B: Q24.1 (B), R222.2 (pin2)
- no-connect marks 37 -> 32
Other:
- note added: "MCU: ESP32-S3-MINI-1 (bottom, antenna at the +x edge)"
- note added: "USB-C PD input (bottom)"
- note added: "front panel (top)"
- note added: "logic supplies: 5 V buck + 3.3 V LDO (bottom)"
- note added: "output channels (bottom)"
- note removed: "MCU: ESP32-S3-MINI-1"
- note removed: "USB-C PD input"
- note removed: "front panel: OLED + encoder modules"
- note removed: "logic supplies: 5 V buck + 3.3 V LDO"
- note removed: "output channels"
- moved on the sheet: C1, C10, C101, C102, C103, C104, C105, C106, C107, C108, C109, C11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
